File: board/AudioProcessor.brd (EAGLE design)
At the start: 49.5 x 45.7 mm, 47 parts, among them IC1 ATTINY24/44/84-SSU, IC2 LP2951, IC3 LP2951, IC4 TDA7439DS, J1 PINHD-1X3-JST-PH, J2 PINHD-1X3-JST-PH, J3 PINHD-1X3-JST-PH, J4 PINHD-1X3-JST-PH, J5 PINHD-1X3-JST-PH, J6 PINHD-1X6-JST-PH

Commit message: Fix JST header orientation
Connections:
- removed net SHUTDOWN: IC3.3, J5.3
- net +3V3: now also J1.3, J2.3, J3.3, J4.3; no longer J1.1, J2.1, J3.1, J4.1
- net BASS: now also J4.1; no longer J4.3
- net GND: now also IC3.3
- net L-IN-RAW: now also J6.1; no longer J6.6
- net L-OUT: now also J6.2; no longer J6.5
- net MID: now also J3.1; no longer J3.3
- net R-IN-RAW: now also J6.6; no longer J6.1
- net R-OUT: now also J6.5; no longer J6.2
- net TREBLE: now also J2.1; no longer J2.3
- net VCC: now also J5.3; no longer J5.1
- net VOLUME: now also J1.1; no longer J1.3
Routing:
- net SHUTDOWN: track 13.1 -> 0.00 mm
Changed lines of the file:
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@@
 <drawing>
 <settings>
+<setting alwaysvectorfont="no"/>
+<setting keepoldvectorfont="yes"/>
+<setting verticaltext="up"/>
 </settings>
 <grid distance="0.05" unitdist="inch" unit="inch" style="dots" multiple="1" display="yes" altdistance="0.025" altunitdist="inch" altunit="inch"/>
@@
 <wire x1="31.115" y1="24.98" x2="29.63" y2="23.495" width="0.254" layer="1"/>
 <wire x1="29.63" y1="23.495" x2="28.5242" y2="23.495" width="0.254" layer="1"/>
+<contactref element="IC3" pad="3"/>
+<wire x1="35.0266" y1="22.225" x2="35.0266" y2="23.495" width="0" layer="19" extent="1-1"/>
 </signal>
 <signal name="N$3">
@@
 <signal name="L-OUT">
 <contactref element="IC4" pad="27"/>
-<contactref element="J6" pad="5"/>
+<contactref element="J6" pad="2"/>
 <wire x1="28.5242" y1="26.035" x2="24.765" y2="26.035" width="0.254" layer="1"/>
 <wire x1="24.765" y1="26.035" x2="21.59" y2="29.21" width="0.254" layer="1"/>
@@
 <signal name="R-OUT">
 <contactref element="IC4" pad="26"/>
-<contactref element="J6" pad="2"/>
+<contactref element="J6" pad="5"/>
 <wire x1="28.5242" y1="24.765" x2="24.765" y2="24.765" width="0.254" layer="1"/>
 <wire x1="24.765" y1="24.765" x2="20.955" y2="28.575" width="0.254" layer="1"/>
@@
 <contactref element="R5" pad="2"/>
 <contactref element="R3" pad="1"/>
-<contactref element="J1" pad="1"/>
-<contactref element="J2" pad="1"/>
-<contactref element="J3" pad="1"/>
-<contactref element="J4" pad="1"/>
+<contactref element="J1" pad="3"/>
+<contactref element="J2" pad="3"/>
+<contactref element="J3" pad="3"/>
+<contactref element="J4" pad="3"/>
 <wire x1="44.45" y1="32.385" x2="44.45" y2="32.89" width="0.254" layer="1"/>
 <wire x1="33.02" y1="34.925" x2="31.75" y2="36.195" width="0.254" layer="1"/>
@@
 <signal name="L-IN-RAW">
 <contactref element="C7" pad="1"/>
-<contactref element="J6" pad="6"/>
+<contactref element="J6" pad="1"/>
 <wire x1="8.89" y1="15.24" x2="3.89" y2="15.24" width="0.254" layer="1"/>
 <wire x1="3.89" y1="15.24" x2="3.81" y2="15.32" width="0.254" layer="1"/>
@@
 <signal name="R-IN-RAW">
 <contactref element="C4" pad="1"/>
-<contactref element="J6" pad="1"/>
+<contactref element="J6" pad="6"/>
 <wire x1="8.89" y1="25.4" x2="3.89" y2="25.4" width="0.254" layer="1"/>
 <wire x1="3.89" y1="25.4" x2="3.81" y2="25.32" width="0.254" layer="1"/>
@@
 </signal>
 <signal name="VCC">
-<contactref element="J5" pad="1"/>
+<contactref element="J5" pad="3"/>
 <contactref element="D2" pad="1"/>
 <wire x1="45.72" y1="25.305" x2="45.72" y2="21.727" width="0.762" layer="1"/>
@@
 <signal name="VOLUME">
 <contactref element="IC1" pad="13"/>
-<contactref element="J1" pad="3"/>
+<contactref element="J1" pad="1"/>
 <wire x1="8.89" y1="37.3634" x2="8.89" y2="41.37" width="0.254" layer="1"/>
 <wire x1="8.89" y1="41.37" x2="9.43" y2="41.91" width="0.254" layer="1"/>
@@
 <signal name="TREBLE">
 <contactref element="IC1" pad="12"/>
-<contactref element="J2" pad="3"/>
+<contactref element="J2" pad="1"/>
 <wire x1="10.16" y1="39.37" x2="10.795" y2="40.005" width="0.254" layer="1"/>
 <wire x1="10.16" y1="39.37" x2="10.16" y2="37.3634" width="0.254" layer="1"/>
@@
 <signal name="MID">
 <contactref element="IC1" pad="11"/>
-<contactref element="J3" pad="3"/>
+<contactref element="J3" pad="1"/>
 <wire x1="12.7" y1="39.37" x2="25.4" y2="39.37" width="0.254" layer="1"/>
 <wire x1="12.7" y1="39.37" x2="11.43" y2="38.1" width="0.254" layer="1"/>
@@
 <signal name="BASS">
 <contactref element="IC1" pad="10"/>
-<contactref element="J4" pad="3"/>
+<contactref element="J4" pad="1"/>
 <wire x1="13.335" y1="38.735" x2="33.655" y2="38.735" width="0.254" layer="1"/>
 <wire x1="13.335" y1="38.735" x2="12.7" y2="38.1" width="0.254" layer="1"/>
@@
 <wire x1="36.1" y1="41.18" x2="36.1" y2="41.91" width="0.254" layer="1"/>
 </signal>
-<signal name="SHUTDOWN">
-<contactref element="IC3" pad="3"/>
-<contactref element="J5" pad="3"/>
-<wire x1="45.72" y1="29.305" x2="43.275" y2="29.305" width="0.254" layer="1"/>
-<wire x1="41.275" y1="27.305" x2="40.005" y2="27.305" width="0.254" layer="1"/>
-<wire x1="36.195" y1="23.495" x2="35.0266" y2="23.495" width="0.254" layer="1"/>
-<wire x1="43.275" y1="29.305" x2="41.275" y2="27.305" width="0.254" layer="1"/>
-<wire x1="40.005" y1="27.305" x2="36.195" y2="23.495" width="0.254" layer="1"/>
-</signal>
 <signal name="N$2">

Commit message: Board updates for manufacturing
Parts:
- J5: value PINHD-1X3-JST-PH -> PINHD-1X2-JST-PH; device SaintGimp:JST-B3B-PH -> SaintGimp:JST-B2B-PH
Connections:
- net GND: now also J5.1; no longer J5.2
- net VCC: now also J5.2; no longer J5.3
Routing:
- net GND: track 39.9 -> 41.2 mm
- net VCC: track 3.58 -> 4.58 mm
Other:
- board text removed: "SHUTDN"
Changed lines of the file:
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@@
 <drawing>
 <settings>
-<setting alwaysvectorfont="no"/>
-<setting keepoldvectorfont="yes"/>
-<setting verticaltext="up"/>
 </settings>
 <grid distance="0.05" unitdist="inch" unit="inch" style="dots" multiple="1" display="yes" altdistance="0.025" altunitdist="inch" altunit="inch"/>
@@
 <text x="35.56" y="44.45" size="0.8128" layer="22" rot="SMR180" align="top-center">LVL</text>
 <text x="38.1" y="44.45" size="0.8128" layer="22" rot="SMR180" align="top-center">GND</text>
-<text x="48.26" y="21.844" size="0.8128" layer="22" rot="SMR270" align="top-center">VIN 10-16V</text>
-<text x="48.26" y="27.305" size="0.8128" layer="22" rot="SMR270" align="top-center">GND</text>
-<text x="48.26" y="31.496" size="0.8128" layer="22" rot="SMR270" align="top-center">SHUTDN</text>
+<text x="48.26" y="23.749" size="0.8128" layer="22" rot="SMR270" align="top-center">VIN 10-16V</text>
+<text x="48.26" y="29.21" size="0.8128" layer="22" rot="SMR270" align="top-center">GND</text>
 <text x="1.27" y="27.051" size="0.8128" layer="22" rot="SMR90" align="top-center">RIN</text>
 <text x="1.27" y="23.876" size="0.8128" layer="22" rot="SMR90" align="top-center">ROUT</text>
@@
 <attribute name="NAME" x="41.656" y="17.9705" size="0.8128" layer="25" rot="R180"/>
 </element>
-<element name="J5" library="SaintGimp" package="JST-B3B-PH" value="PINHD-1X3-JST-PH" x="45.72" y="27.305" smashed="yes" rot="R90">
+<element name="J5" library="SaintGimp" package="JST-B2B-PH" value="PINHD-1X2-JST-PH" x="45.72" y="27.305" smashed="yes" rot="R90">
 <attribute name="NAME" x="43.1830625" y="31.01715" size="0.8128" layer="25" ratio="10" rot="R180"/>
 </element>
@@
 <contactref element="J3" pad="2"/>
 <contactref element="J4" pad="2"/>
-<contactref element="J5" pad="2"/>
+<contactref element="J5" pad="1"/>
 <polygon width="0.4064" layer="16">
 <vertex x="0" y="45.72"/>
@@
 <wire x1="39.5" y1="29.21" x2="41.275" y2="29.21" width="0.254" layer="1"/>
 <via x="34.29" y="20.955" extent="1-16" drill="0.5"/>
-<wire x1="35.0266" y1="22.225" x2="35.0266" y2="21.6916" width="0.254" layer="1"/>
+<wire x1="35.0266" y1="21.6916" x2="35.0266" y2="22.225" width="0.254" layer="1"/>
 <wire x1="35.0266" y1="21.6916" x2="34.29" y2="20.955" width="0.254" layer="1"/>
 <wire x1="16.399" y1="7.985" x2="15.875" y2="7.985" width="0.254" layer="1"/>
@@
 <wire x1="29.63" y1="23.495" x2="28.5242" y2="23.495" width="0.254" layer="1"/>
 <contactref element="IC3" pad="3"/>
-<wire x1="35.0266" y1="22.225" x2="35.0266" y2="23.495" width="0" layer="19" extent="1-1"/>
+<wire x1="35.0266" y1="22.225" x2="35.0266" y2="23.495" width="0.254" layer="1"/>
 </signal>
 <signal name="N$3">
@@
 </signal>
 <signal name="VCC">
-<contactref element="J5" pad="3"/>
+<contactref element="J5" pad="2"/>
 <contactref element="D2" pad="1"/>
-<wire x1="45.72" y1="25.305" x2="45.72" y2="21.727" width="0.762" layer="1"/>
+<wire x1="45.72" y1="21.727" x2="45.72" y2="26.305" width="0.762" layer="1"/>
 </signal>
 <signal name="N$19">
